File: Kicad/RC/RC.kicad_sch (KiCad schematic)
At the start: 4 parts, among them SW1 SW_Push, SW2 SW_Wuerth_450301014042

Commit message: update SW1 footprint
Parts:
- SW1: footprint Button_Switch_THT:SW_Push_2P1T_Toggle_CK_PVA1xxH1xxxxxxV2 -> SamacSys_Parts:SW_Push_2P1T_Toggle_CK_PVA1xxH1xxxxxxV3
Changed lines of the file:
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@@
 			)
 		)
-		(property "Footprint" "Button_Switch_THT:SW_Push_2P1T_Toggle_CK_PVA1xxH1xxxxxxV2"
+		(property "Footprint" "SamacSys_Parts:SW_Push_2P1T_Toggle_CK_PVA1xxH1xxxxxxV3"
 			(at 116.84 77.47 0)
 			(effects
